File: hardware/board/butns.kicad_pcb (KiCad board)
At the start: 2 copper layers, 99 x 99 mm, 265 parts, among them J1 Conn_01x08, SW1 SW_Push, SW10 SW_Push, SW11 SW_Push, SW12 SW_Push, SW13 SW_Push, SW14 SW_Push, SW15 SW_Push, SW16 SW_Push, SW17 SW_Push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

Commit message: Remove Buttons Silkscreen name, update version
Other:
- board text added: "v2 2025"
- board text removed: "v0.1 2024"
